Commit message: feat(urdf): 更新 tip link

File: src/tomato_picker/description/urdf/tomato_picker.urdf (robot description, URDF)
Before this commit: robot Tomato-Picker, 11 links, 10 joints
Links:
- added link tip
- link Link6: mass 0.774251897736 -> 0.785649631359557
Joints:
- added joint tip_joint: type fixed, parent tool0, child tip, origin xyz=0 0 0.101 rpy=0 0 0
